File: sch/gp-ctrl.kicad_pcb (KiCad board)
At the start: 2 copper layers, 65 x 56.5 mm, 128 parts, among them J1 DNP, J10 3.5mm, J11 3.5mm, J12 3.5mm, J13 3.5mm, J14 DNP, J15 DNP, J16 Conn_02x06_Odd_Even, J17 USB_B_Micro, J18 DNF, J19 Screw_Terminal_3.5mm, J20 Screw_Terminal_3.5mm, J3 Conn_02x20_Odd_Even, J4 Screw_Terminal_3.5mm, J5 2.54mm, J6 2.54mm, J7 2.54mm, J8 DNP, J9 2.54mm, K1 Relay_DPDT_Panasonic_AGQ200A4H, K2 Relay_DPDT_Panasonic_AGQ200A4H, Q1 2N7002P, Q10 2N7002P, Q11 2N7002P, Q12 2N7002P, Q2 IRLML6244, Q3 2N7002P, Q4 IRLML6244, Q5 2N7002P, Q6 2N7002P, Q7 2N7002P, Q8 2N7002P, Q9 2N7002P, SW1 C2689642, SW2 C2689642, SW3 C2689642, U1 INA219AxD, U2 W25Q64JVSSIQ, U3 RP2040, U4 NCP1117LPST33T3G, U5 MP1584EN-LF-Z, Y1 12MHz

Commit message: updated pcb
Parts:
- moved C9 66.8 mm to (177.3, 126.1), turned to 90 degrees
- moved C12 62.7 mm to (164.8, 126.2), turned to 180 degrees
- moved C13 60.9 mm to (164.8, 127.2), turned to 180 degrees
- moved C8 59.9 mm to (172.8, 134.2)
- moved C15 58.6 mm to (170.4, 136.3), turned to -90 degrees
- moved C4 58.0 mm to (176.3, 126.4), turned to 90 degrees
- moved C14 56.3 mm to (171.4, 136.3), turned to -90 degrees
- moved C11 47.2 mm to (169.2, 123.3), turned to 90 degrees
- moved C10 46.9 mm to (172.3, 122.9), turned to 90 degrees
- moved C6 44.5 mm to (164.8, 128.2), turned to 180 degrees
- moved C5 44.4 mm to (164.8, 125.2), turned to 180 degrees
- moved C7 43.2 mm to (164.8, 129.2), turned to 180 degrees
- moved J18 17.1 mm to (178.2, 122.2)
- moved C3 14.7 mm to (164.3, 130.2), turned to 180 degrees
- moved R32 11.4 mm to (163.7, 131.6), turned to 180 degrees
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Routing:
- net +3V3: track 0.00 -> 26.0 mm
- net +1V1: track 0.00 -> 7.92 mm
